File: solorCharger.sch (KiCad schematic (older format))
At the start: 31 parts

Commit message: MPPT設定
Parts:
- added R?: 1k, symbol R
- added U?: LM234, symbol LM234
- D? (x2): symbol LED -> LED-RESCUE-solorCharger
- R?: value R -> 390k
- R?: value R -> 15k
- R?: value R -> 40m
Connections:
- net at R?.1, R?.2, U?.2 (MPPSET): now also R?.2, U?.3 (V-)
- net at D?.2 (A), J?.2 (P2), R?.1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: now also U?.1 (V+)
- new net: R?.1, U?.2 (R)
Changed lines of the file:
@@
 EESchema Schematic File Version 2
+LIBS:solorCharger-rescue
 LIBS:power
 LIBS:device
@@
 LIBS:valves
 LIBS:KiCADKozueLib
+LIBS:solorCharger-cache
 EELAYER 25 0
 EELAYER END
@@
 $EndComp
 $Comp
-L LED D?
+L LED-RESCUE-solorCharger D?
 U 1 1 58BF8D6E
 P 3800 5150
@@
 $EndComp
 $Comp
-L LED D?
+L LED-RESCUE-solorCharger D?
 U 1 1 58BF8DBD
 P 3800 5450
@@
 P 3650 3550
 F 0 "R?" V 3730 3550 50  0000 C CNN
-F 1 "R" V 3650 3550 50  0000 C CNN
+F 1 "390k" V 3650 3550 50  0000 C CNN
 F 2 "" V 3580 3550 50  0000 C CNN
 F 3 "" H 3650 3550 50  0000 C CNN
@@
 P 3650 4150
 F 0 "R?" V 3730 4150 50  0000 C CNN
-F 1 "R" V 3650 4150 50  0000 C CNN
+F 1 "15k" V 3650 4150 50  0000 C CNN
 F 2 "" V 3580 4150 50  0000 C CNN
 F 3 "" H 3650 4150 50  0000 C CNN
@@
 P 7400 4450
 F 0 "R?" V 7480 4450 50  0000 C CNN
-F 1 "R" V 7400 4450 50  0000 C CNN
+F 1 "40m" V 7400 4450 50  0000 C CNN
 F 2 "" V 7330 4450 50  0000 C CNN
 F 3 "" H 7400 4450 50  0000 C CNN
@@
 	3650 4300 3650 4350
 Wire Wire Line
-	3650 3850 4500 3850
+	3050 3850 4500 3850
 Connection ~ 3650 3850
 Wire Wire Line
@@
 	2600 5450 3250 5450
 Connection ~ 2600 5150
+$Comp
+L LM234 U?
+U 1 1 58D0021C
+P 3050 2950
+F 0 "U?" H 2800 3000 60  0000 C CNN
+F 1 "LM234" H 2800 2900 60  0000 C CNN
+F 2 "" H 3050 2950 60  0001 C CNN
+F 3 "" H 3050 2950 60  0001 C CNN
+	1    3050 2950
+	1    0    0    -1
+$EndComp
+$Comp
+L R R?
+U 1 1 58D00769
+P 3450 3550
+F 0 "R?" V 3530 3550 50  0000 C CNN
+F 1 "1k" V 3450 3550 50  0000 C CNN
+F 2 "" V 3380 3550 50  0000 C CNN
+F 3 "" H 3450 3550 50  0000 C CNN
+	1    3450 3550
+	1    0    0    -1
+$EndComp
+Wire Wire Line
+	3450 2950 3450 3400
+Wire Wire Line
+	3450 3850 3450 3700
+Wire Wire Line
+	3050 3400 3050 3850
+Connection ~ 3450 3850
+Connection ~ 3050 2500
 $EndSCHEMATC
